Commit message: feat: add controls to the robots

File: src/my_robot/urdf/robot4.urdf (robot description, URDF)
Before this commit: robot ${robot_name}, 3 links, 2 joints
Links:
- removed link ${robot_name}_base_link
- removed link ${robot_name}_left_wheel
- removed link ${robot_name}_right_wheel
- added link robot4_base_link, mass 5; collision cylinder length=0.1 radius=0.2; visual cylinder length=0.1 radius=0.2
- added link robot4_left_wheel, mass 1; collision cylinder length=0.05 radius=0.05; visual cylinder length=0.05 radius=0.05
- added link robot4_right_wheel, mass 1; collision cylinder length=0.05 radius=0.05; visual cylinder length=0.05 radius=0.05
Joints:
- removed joint ${robot_name}_left_wheel_joint
- removed joint ${robot_name}_right_wheel_joint
- added joint robot4_left_wheel_joint: type continuous, parent robot4_base_link, child robot4_left_wheel, origin xyz=0 0.15 -0.05 rpy=1.5708 0 0, axis 0 0 1
- added joint robot4_right_wheel_joint: type continuous, parent robot4_base_link, child robot4_right_wheel, origin xyz=0 -0.15 -0.05 rpy=1.5708 0 0, axis 0 0 1

File: src/my_robot/urdf/robot5.urdf (robot description, URDF)
Before this commit: robot ${robot_name}, 3 links, 2 joints
Links:
- removed link ${robot_name}_base_link
- removed link ${robot_name}_left_wheel
- removed link ${robot_name}_right_wheel
- added link robot5_base_link, mass 5; collision cylinder length=0.1 radius=0.2; visual cylinder length=0.1 radius=0.2
- added link robot5_left_wheel, mass 1; collision cylinder length=0.05 radius=0.05; visual cylinder length=0.05 radius=0.05
- added link robot5_right_wheel, mass 1; collision cylinder length=0.05 radius=0.05; visual cylinder length=0.05 radius=0.05
Joints:
- removed joint ${robot_name}_left_wheel_joint
- removed joint ${robot_name}_right_wheel_joint
- added joint robot5_left_wheel_joint: type continuous, parent robot5_base_link, child robot5_left_wheel, origin xyz=0 0.15 -0.05 rpy=1.5708 0 0, axis 0 0 1
- added joint robot5_right_wheel_joint: type continuous, parent robot5_base_link, child robot5_right_wheel, origin xyz=0 -0.15 -0.05 rpy=1.5708 0 0, axis 0 0 1

File: src/my_robot/urdf/robot6.urdf (robot description, URDF)
Before this commit: robot ${robot_name}, 3 links, 2 joints
Links:
- removed link ${robot_name}_base_link
- removed link ${robot_name}_left_wheel
- removed link ${robot_name}_right_wheel
- added link robot6_base_link, mass 5; collision cylinder length=0.1 radius=0.2; visual cylinder length=0.1 radius=0.2
- added link robot6_left_wheel, mass 1; collision cylinder length=0.05 radius=0.05; visual cylinder length=0.05 radius=0.05
- added link robot6_right_wheel, mass 1; collision cylinder length=0.05 radius=0.05; visual cylinder length=0.05 radius=0.05
Joints:
- removed joint ${robot_name}_left_wheel_joint
- removed joint ${robot_name}_right_wheel_joint
- added joint robot6_left_wheel_joint: type continuous, parent robot6_base_link, child robot6_left_wheel, origin xyz=0 0.15 -0.05 rpy=1.5708 0 0, axis 0 0 1
- added joint robot6_right_wheel_joint: type continuous, parent robot6_base_link, child robot6_right_wheel, origin xyz=0 -0.15 -0.05 rpy=1.5708 0 0, axis 0 0 1

File: src/my_robot/urdf/robot7.urdf (robot description, URDF)
Before this commit: robot ${robot_name}, 3 links, 2 joints
Links:
- removed link ${robot_name}_base_link
- removed link ${robot_name}_left_wheel
- removed link ${robot_name}_right_wheel
- added link robot7_base_link, mass 5; collision cylinder length=0.1 radius=0.2; visual cylinder length=0.1 radius=0.2
- added link robot7_left_wheel, mass 1; collision cylinder length=0.05 radius=0.05; visual cylinder length=0.05 radius=0.05
- added link robot7_right_wheel, mass 1; collision cylinder length=0.05 radius=0.05; visual cylinder length=0.05 radius=0.05
Joints:
- removed joint ${robot_name}_left_wheel_joint
- removed joint ${robot_name}_right_wheel_joint
- added joint robot7_left_wheel_joint: type continuous, parent robot7_base_link, child robot7_left_wheel, origin xyz=0 0.15 -0.05 rpy=1.5708 0 0, axis 0 0 1
- added joint robot7_right_wheel_joint: type continuous, parent robot7_base_link, child robot7_right_wheel, origin xyz=0 -0.15 -0.05 rpy=1.5708 0 0, axis 0 0 1
