Commit message: feat: add object avoidance controller

File: src/my_robot/urdf/robot1.urdf (robot description, URDF)
Before this commit: robot robot1, 4 links, 3 joints
Joints:
- joint robot1_camera_joint: origin xyz=0 0 0.35 rpy=0 0 0 -> xyz=0.2 0 0.15 rpy=0 -1.5708 0

File: src/my_robot/urdf/robot2.urdf (robot description, URDF)
Before this commit: robot robot2, 4 links, 3 joints
Joints:
- joint robot2_camera_joint: origin xyz=0 0 0.35 rpy=0 0 0 -> xyz=0.2 0 0.15 rpy=0 -1.5708 0

File: src/my_robot/urdf/robot3.urdf (robot description, URDF)
Before this commit: robot robot3, 4 links, 3 joints
Joints:
- joint robot3_camera_joint: origin xyz=0 0 0.35 rpy=0 0 0 -> xyz=0.2 0 0.15 rpy=0 -1.5708 0
